File: hardware/power_usb.kicad_sch (KiCad schematic)
At the start: 0 parts

Commit message: Fix Power & USB sheet wiring, footprints and annotation
- Ground regulator U202 pin 2 (was unconnected)
- Shield network R203 || C201 to GND (was in series)
- D202 Schottky anode on VBUS_FUSED (was reversed)
- D201 as unidirectional TVS, cathode on VBUS_FUSED
- Correct footprints on all parts; DNP attribute on C202, D202
- Power symbols for GND/VBUS rails, PWR_FLAGs, local VBUS_FUSED label
- Symbol instances moved to the gps-lora project hierarchy

Co-Authored-By: Claude Opus 5.5 <noreply@anthropic.com>
Parts:
- added C201: 4.7nF, Capacitor_SMD:C_0402_1005Metric, symbol Device:C
- added C202: 2200uF, Capacitor_SMD:CP_Elec_10x10.5, symbol Device:C_Polarized
- added C203, C205: 22uF, Capacitor_SMD:C_0805_2012Metric, symbol Device:C
- added C204, C206: 100nF, Capacitor_SMD:C_0402_1005Metric, symbol Device:C
- added D201: 5V TVS, Diode_SMD:D_SOD-123F, symbol Device:D_Zener
- added D202: Schottky, Diode_SMD:D_SMA, symbol Device:D_Schottky
- added F201: 750mA, Fuse:Fuse_1206_3216Metric, symbol Device:Polyfuse
- added J201: TYPE-C-31-M-12, Connector_USB:USB_C_Receptacle_HRO_TYPE-C-31-M-12, symbol Connector:USB_C_Receptacle_USB2.0_16P
- added R201, R202: 5.1k, Resistor_SMD:R_0402_1005Metric, symbol Device:R
- added R203: 1M, Resistor_SMD:R_0402_1005Metric, symbol Device:R
- added R204: 0R, Resistor_SMD:R_0805_2012Metric, symbol Device:R
- added R205: 10k, Resistor_SMD:R_0402_1005Metric, symbol Device:R
- added R206: 15k, Resistor_SMD:R_0402_1005Metric, symbol Device:R
- added TP201, TP202, TP203, TP204: TestPoint, TestPoint:TestPoint_Pad_D1.0mm, symbol Connector:TestPoint
- added U201: USBLC6-2SC6, Package_TO_SOT_SMD:SOT-23-6, symbol Power_Protection:USBLC6-2SC6
- added U202: AP7361C-33E, Package_TO_SOT_SMD:SOT-223-3_TabPin2, symbol Regulator_Linear:AP7361C-33E
Connections:
- new net: C201.1, J201.SH (SHIELD), R203.1
- new net: J201.A5 (CC1), R201.1
- new net: J201.B5 (CC2), R202.1
- new net +3V3: C205.1, C206.1, TP203.1, U202.3 (VO)
- new net +5V: C202.1, C203.1, C204.1, D202.1 (K), R204.2, U202.1 (VI)
- new net GND: C201.2, C202.2, C203.2, C204.2, C205.2, C206.2, D201.2 (A), J201.A1 (GND), J201.A12 (GND), J201.B1 (GND), J201.B12 (GND), R201.2, R202.2, R203.2, R206.2, TP204.1, U201.2 (GND), U202.2 (GND)
- new net USB_DN: J201.A7 (D-), J201.B7 (D-), U201.3 (I/O2), U201.4 (I/O2)
- new net USB_DP: J201.A6 (D+), J201.B6 (D+), U201.1 (I/O1), U201.6 (I/O1)
- new net VBUS: F201.1, J201.A4 (VBUS), J201.A9 (VBUS), J201.B4 (VBUS), J201.B9 (VBUS), R205.1, TP201.1, U201.5 (VBUS)
- new net VBUS_FUSED: D201.1 (K), D202.2 (A), F201.2, R204.1, TP202.1
- new net VBUS_SENSE: R205.2, R206.1
- no-connect marks 0 -> 2

Commit message: Complete schematic, place and partially route the PCB
Schematic:
- Add Storage & Display sheet (microSD, FH12 OLED connector, TLV75801
  3.8 V VBAT regulator, charge-pump parts) and Radio sheet fixes
- Select remaining parts (PTS810, 1206L075THYR, SMF5.0A, MCP120 EN
  supervisor DNP, Elna DSK backup cap), add mounting holes and fiducials
- Pin changes for routability: PPS -> IO15, LoRa MOSI -> IO47,
  LoRa RESET -> IO48, LoRa DIO0 -> IO1
- Remove optional SPI clock filter parts (R309/C307, R310/C308)
- Remove company name from title blocks (personal project)

PCB (60 x 120 mm, 4 layers):
- Place all parts; GNSS zone with custom DRC rules (kicad_dru)
- Project ESP32-S3-WROOM-1 footprint with 0.4 mm thermal vias
- GND / +3V3 / +5V copper zones
- Route power path, GNSS, microSD and LoRa buses
- DRC clean except unrouted nets and expected silkscreen-at-edge items

Docs: selected-parts table, pin table and EMC deviation in PCB_DESIGN.md

Co-Authored-By: Claude Opus 5.5 <noreply@anthropic.com>
Parts:
- D201: value 5V TVS -> SMF5.0A
- F201: value 750mA -> 0.75A PTC
Other:
- company: SSS-Defence -> (none)
Changed lines of the file:
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@@
 		(date "2026-10-05")
 		(rev "v0.1")
-		(company "SSS-Defence")
 		(comment 1 "CERN-OHL-P-2.0")
 		(comment 2 "https://github.com/Majorwhiskey/gps-lora")
@@
 			)
 		)
-		(property "Value" "750mA"
+		(property "Value" "0.75A PTC"
 			(at 91.44 77.47 90)
 			(show_name no)
@@
 			)
 		)
-		(property "Value" "5V TVS"
+		(property "Value" "SMF5.0A"
 			(at 91.44 93.9799 90)
 			(show_name no)

Commit message: Finish PCB routing, add BOM part numbers and fab export
Routing (DRC: 0 errors, 0 unconnected; ERC: 0)
- Complete the remaining nets on top of the GUI routing; GND stitching
  grid and edge fence; every GND pad reaches the L2 plane
- Re-lay the microSD bus under USB D+ so the USBLC6 and VBUS TVS get
  direct GND vias; lift LoRa NSS/MISO/MOSI to clear the TVS via
- Reroute D-, VBUS sense, CC2, BOOT, OLED SDA/SCL, LED and TXD0_R; remove
  vias in pads (R205, R505, R204, R507, U301 pin 7)
- Placement tweaks: C306 moved, C508/C509/R508 rotated 180, R302 moved
- PCB title block with rev v0.1

Parts and outputs
- MPN and Manufacturer fields on all placed parts (tools/add-mpn.py)
- tools/fab-export.py: ERC/DRC gate, zone refill, Gerbers, drill, BOM,
  pick-and-place and fab notes for Lion Circuits
- OLED panel DS501: schematic symbol and board-only 3D footprint
- Elna DSK footprint for C403 (not placed yet)
- kicad-routing skill under .claude/skills

Open before fab (see docs/PCB_DESIGN.md Open items): J502 pin order is
mirrored against the panel FPC; Lion stackup widths; C403 placement.

Co-Authored-By: Claude Opus 5.5 <noreply@anthropic.com>
Parts:
- C201: MPN (none) -> GRM155R71H472KA01D; Manufacturer (none) -> Murata
- C203, C205: MPN (none) -> CL21A226MAQNNNE; Manufacturer (none) -> Samsung
- C204, C206: MPN (none) -> CL05B104KO5NNNC; Manufacturer (none) -> Samsung
- D201: MPN (none) -> SMF5.0A; Manufacturer (none) -> Littelfuse
- D202: MPN (none) -> B340A-13-F; Manufacturer (none) -> Diodes Inc
- F201: MPN (none) -> 1206L075THYR; Manufacturer (none) -> Littelfuse
- J201: MPN (none) -> TYPE-C-31-M-12; Manufacturer (none) -> Korean Hroparts (HRO)
- R201, R202: MPN (none) -> RC0402FR-075K1L; Manufacturer (none) -> Yageo
- R203: MPN (none) -> RC0402FR-071ML; Manufacturer (none) -> Yageo
- R204: MPN (none) -> RC0805JR-070RL; Manufacturer (none) -> Yageo
- R205: MPN (none) -> RC0402FR-0710KL; Manufacturer (none) -> Yageo
- R206: MPN (none) -> RC0402FR-0715KL; Manufacturer (none) -> Yageo
- U201: MPN (none) -> USBLC6-2SC6; Manufacturer (none) -> STMicroelectronics
- U202: MPN (none) -> AP7361C-33E-13; Manufacturer (none) -> Diodes Inc
