File: hardware/theoros.kicad_sch (KiCad schematic)
At the start: 7 parts

Commit message: Rename project to Theoros and add V1.0 silkscreen artwork
Theoros (Greek θεωρός): an official observer and envoy, sent to watch
and report back.

Rename gps-lora to theoros everywhere: KiCad project, symbol and
footprint libraries, firmware library (theoros-core), umbrella header,
PC tool (tools/theoros.py), NVS namespaces, mDNS hostname, docs and
title blocks. The HKDF salt is now "theoros" (7 bytes), so every derived
key changes; the SECURITY.md test vectors are recomputed and host tests
pass. Boards provisioned with the old salt need re-provisioning.

Board revision is now V1.0. Silkscreen additions:
- Top: "THEOROS ${REVISION}" and "ΘΕΩΡΟΣ", an antenna warning next to
  J401, and a hidden line under the OLED panel.
- Bottom: an owl made as a solder-mask opening over the GND pour (gold
  with ENIG; vias inside stay tented) and the motto "ΟΡΩ ΚΑΙ ΑΓΓΕΛΛΩ /
  I SEE AND I REPORT".
Fab notes now state silkscreen on both sides and the intentional mask
opening. DRC is unchanged from before (4 silk-edge warnings).

Co-Authored-By: Claude Opus 5.5 <noreply@anthropic.com>
Other:
- title: GPS LoRa Logger -> Theoros
Changed lines of the file:
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@@
 	(paper "A4")
 	(title_block
-		(title "GPS LoRa Logger")
+		(title "Theoros")
 		(date "2026-10-05")
-		(rev "v0.1")
+		(rev "V1.0")
 		(comment 1 "CERN-OHL-P-2.0")
-		(comment 2 "https://github.com/Majorwhiskey/gps-lora")
+		(comment 2 "https://github.com/Majorwhiskey/theoros")
 	)
 	(symbol
@@
 		)
 		(instances
-			(project "gps-lora"
+			(project "theoros"
 				(path "/4fe56230-194d-489d-a2bc-70162e8e6b48"
 					(reference "FID3")
@@
 		)
 		(instances
-			(project "gps-lora"
+			(project "theoros"
 				(path "/4fe56230-194d-489d-a2bc-70162e8e6b48"
 					(reference "#PWR052")
@@
 		)
 		(instances
-			(project "gps-lora"
+			(project "theoros"
 				(path "/4fe56230-194d-489d-a2bc-70162e8e6b48"
 					(reference "#PWR030")
@@
 		)
 		(instances
-			(project "gps-lora"
+			(project "theoros"
 				(path "/4fe56230-194d-489d-a2bc-70162e8e6b48"
 					(reference "H1")
@@
 		)
 		(instances
-			(project "gps-lora"
+			(project "theoros"
 				(path "/4fe56230-194d-489d-a2bc-70162e8e6b48"
 					(reference "H2")
@@
 		)
 		(instances
-			(project "gps-lora"
+			(project "theoros"
 				(path "/4fe56230-194d-489d-a2bc-70162e8e6b48"
 					(reference "#PWR049")
@@
 		)
 		(instances
-			(project "gps-lora"
+			(project "theoros"
 				(path "/4fe56230-194d-489d-a2bc-70162e8e6b48"
 					(reference "FID1")
@@
 		)
 		(instances
-			(project "gps-lora"
+			(project "theoros"
 				(path "/4fe56230-194d-489d-a2bc-70162e8e6b48"
 					(reference "H3")
@@
 		)
 		(instances
-			(project "gps-lora"
+			(project "theoros"
 				(path "/4fe56230-194d-489d-a2bc-70162e8e6b48"
 					(reference "#PWR048")
@@
 		)
 		(instances
-			(project "gps-lora"
+			(project "theoros"
 				(path "/4fe56230-194d-489d-a2bc-70162e8e6b48"
 					(reference "H4")
@@
 		)
 		(instances
-			(project "gps-lora"
+			(project "theoros"
 				(path "/4fe56230-194d-489d-a2bc-70162e8e6b48"
 					(reference "FID2")
@@
 		)
 		(instances
-			(project "gps-lora"
+			(project "theoros"
 				(path "/4fe56230-194d-489d-a2bc-70162e8e6b48"
 					(page "3")
@@
 		)
 		(instances
-			(project "gps-lora"
+			(project "theoros"
 				(path "/4fe56230-194d-489d-a2bc-70162e8e6b48"
 					(page "5")
@@
 		)
 		(instances
-			(project "gps-lora"
+			(project "theoros"
 				(path "/4fe56230-194d-489d-a2bc-70162e8e6b48"
 					(page "2")
@@
 		)
 		(instances
-			(project "gps-lora"
+			(project "theoros"
 				(path "/4fe56230-194d-489d-a2bc-70162e8e6b48"
 					(page "4")
