File: hardware/radio.kicad_sch (KiCad schematic)
At the start: 0 parts

Commit message: Add Radio sheet
u-blox SAM-M10Q GNSS (pin-compatible SAM-M8Q symbol and footprint,
footprint checked against the integration manual land pattern) with
decoupling, SAFEBOOT test pad and DNP backup-supply network.
HopeRF RFM95W-868S2 with decoupling and Hirose U.FL antenna connector.

Co-Authored-By: Claude Opus 5.5 <noreply@anthropic.com>
Parts:
- added C401, C405: 10uF, Capacitor_SMD:C_0805_2012Metric, symbol Device:C
- added C402, C406: 100nF, Capacitor_SMD:C_0402_1005Metric, symbol Device:C
- added C403: 0.2F supercap, symbol Device:C
- added C404: 100uF, Capacitor_SMD:C_1210_3225Metric, symbol Device:C
- added D401: BAT54, Diode_SMD:D_SOD-323, symbol Device:D_Schottky
- added J401: U.FL, Connector_Coaxial:U.FL_Hirose_U.FL-R-SMT-1_Vertical, symbol Connector:Conn_Coaxial
- added R401: 1k, Resistor_SMD:R_0402_1005Metric, symbol Device:R
- added TP401: SAFEBOOT, TestPoint:TestPoint_Pad_D1.0mm, symbol Connector:TestPoint
- added U401: SAM-M10Q, RF_GPS:ublox_SAM-M8Q, symbol RF_GPS:SAM-M8Q
- added U402: RFM95W-868S2, RF_Module:HOPERF_RFM9XW_SMD, symbol RF_Module:RFM95W-868S2
Connections:
- new net: D401.1 (K), R401.1
- new net +3V3: C401.1, C402.1, C404.1, C405.1, C406.1, D401.2 (A), U401.17 (VCC), U401.2 (VCC_IO), U402.13 (3.3V)
- new net GND: C401.2, C402.2, C403.2, C404.2, C405.2, C406.2, J401.2 (Ext), U401.1 (GND), U401.10 (GND), U401.11 (GND), U401.15 (GND), U401.16 (GND), U401.20 (GND), U401.4 (GND), U401.5 (GND), U401.6 (GND), U402.1 (GND), U402.10 (GND), U402.8 (GND)
- new net GNSS_PPS: U401.7 (TIMEPULSE)
- new net GNSS_RESET_N: U401.18 (~{RESET})
- new net GNSS_RXD: U401.14 (RXD)
- new net GNSS_SAFEBOOT: TP401.1, U401.8 (~{SAFEBOOT})
- new net GNSS_TXD: U401.13 (TXD)
- new net GNSS_VBCKP: C403.1, R401.2, U401.3 (V_BCKP)
- new net LORA_ANT: J401.1 (In), U402.9 (ANT)
- new net LORA_DIO0: U402.14 (DIO0)
- new net LORA_DIO1: U402.15 (DIO1)
- new net LORA_MISO: U402.2 (MISO)
- new net LORA_MOSI: U402.3 (MOSI)
- new net LORA_NSS: U402.5 (NSS)
- new net LORA_RESET: U402.6 (RESET)
- new net LORA_SCK: U402.4 (SCK)
- no-connect marks 0 -> 7
Other:
- note added: "50 ohm microstrip, under 10 mm"
- note added: "GNSS backup option, DNP in v1"
- note added: "GNSS: u-blox SAM-M10Q (pin-compatible with SAM-M8Q symbol/footprint)"
- note added: "LoRa: HopeRF RFM95W-868S2 (order code is mandatory: 433/470/915 variants share the footprint)"
- note added: "No capacitor on RESET, no load on TIMEPULSE (SAFEBOOT strap). V_BCKP open in v1."
- note added: "RESET: drive low or high-Z only. +20 dBm limited to 1% duty cycle."

Commit message: Complete schematic, place and partially route the PCB
Schematic:
- Add Storage & Display sheet (microSD, FH12 OLED connector, TLV75801
  3.8 V VBAT regulator, charge-pump parts) and Radio sheet fixes
- Select remaining parts (PTS810, 1206L075THYR, SMF5.0A, MCP120 EN
  supervisor DNP, Elna DSK backup cap), add mounting holes and fiducials
- Pin changes for routability: PPS -> IO15, LoRa MOSI -> IO47,
  LoRa RESET -> IO48, LoRa DIO0 -> IO1
- Remove optional SPI clock filter parts (R309/C307, R310/C308)
- Remove company name from title blocks (personal project)

PCB (60 x 120 mm, 4 layers):
- Place all parts; GNSS zone with custom DRC rules (kicad_dru)
- Project ESP32-S3-WROOM-1 footprint with 0.4 mm thermal vias
- GND / +3V3 / +5V copper zones
- Route power path, GNSS, microSD and LoRa buses
- DRC clean except unrouted nets and expected silkscreen-at-edge items

Docs: selected-parts table, pin table and EMC deviation in PCB_DESIGN.md

Co-Authored-By: Claude Opus 5.5 <noreply@anthropic.com>
Parts:
- C403: value 0.2F supercap -> 0.22F 3.3V
Other:
- company: SSS-Defence -> (none)

Commit message: Finish PCB routing, add BOM part numbers and fab export
Routing (DRC: 0 errors, 0 unconnected; ERC: 0)
- Complete the remaining nets on top of the GUI routing; GND stitching
  grid and edge fence; every GND pad reaches the L2 plane
- Re-lay the microSD bus under USB D+ so the USBLC6 and VBUS TVS get
  direct GND vias; lift LoRa NSS/MISO/MOSI to clear the TVS via
- Reroute D-, VBUS sense, CC2, BOOT, OLED SDA/SCL, LED and TXD0_R; remove
  vias in pads (R205, R505, R204, R507, U301 pin 7)
- Placement tweaks: C306 moved, C508/C509/R508 rotated 180, R302 moved
- PCB title block with rev v0.1

Parts and outputs
- MPN and Manufacturer fields on all placed parts (tools/add-mpn.py)
- tools/fab-export.py: ERC/DRC gate, zone refill, Gerbers, drill, BOM,
  pick-and-place and fab notes for Lion Circuits
- OLED panel DS501: schematic symbol and board-only 3D footprint
- Elna DSK footprint for C403 (not placed yet)
- kicad-routing skill under .claude/skills

Open before fab (see docs/PCB_DESIGN.md Open items): J502 pin order is
mirrored against the panel FPC; Lion stackup widths; C403 placement.

Co-Authored-By: Claude Opus 5.5 <noreply@anthropic.com>
Parts:
- C401, C405: MPN (none) -> CL21A106KAYNNNE; Manufacturer (none) -> Samsung
- C402, C406: MPN (none) -> CL05B104KO5NNNC; Manufacturer (none) -> Samsung
- C403: MPN (none) -> DSK-3R3H224U-HL; Manufacturer (none) -> Elna
- C404: MPN (none) -> GRM32ER61A107ME20L; Manufacturer (none) -> Murata
- D401: MPN (none) -> BAT54WS-7-F; Manufacturer (none) -> Diodes Inc
- J401: MPN (none) -> U.FL-R-SMT-1(10); Manufacturer (none) -> Hirose
- R401: MPN (none) -> RC0402FR-071KL; Manufacturer (none) -> Yageo
- U401: MPN (none) -> SAM-M10Q-00B; Manufacturer (none) -> u-blox
- U402: MPN (none) -> RFM95W-868S2; Manufacturer (none) -> HopeRF

Commit message: Fix J502 pin mapping, place C403 backup, check stackup impedance
J502: the panel FPC lands mirrored on the 180-degree FH12 (panel pin n on
J502 pin 31-n, per the ER-OLED0.96-1.1W drawing 1.4.1). The J502 symbol is
now mirrored in the schematic and the OLED support row is re-placed in the
new pin order and hand-routed. C305 (DNP) turns horizontal and R302 moves
0.4 mm east to make room.

C403: Seiko CPH3225A 11 mF chip EDLC on V_BCKP (~10 min hot-start
hold-up), with a new footprint from the Seiko drawing (pad 1 = +). D401
and R401, which charge it from 3V3, are now fitted. The unused Elna
footprint is removed.

Stackup: Lion's standard 4-layer 1.6 mm build (2116, 0.12 mm to L2) gives
47-49 ohm on LORA_ANT and 89-100 ohm on the USB pair with the existing
0.2 mm traces, so no impedance-controlled order is needed.

DRC: same 4 silk-edge warnings as before, 0 unconnected, schematic parity
clean. ERC clean.

Co-Authored-By: Claude Opus 5.5 <noreply@anthropic.com>
Parts:
- C403: value 0.22F 3.3V -> 11mF 3.3V; footprint (none) -> theoros:Seiko_CPH3225A; MPN DSK-3R3H224U-HL -> CPH3225A; Manufacturer Elna -> Seiko Instruments; now fitted
- D401, R401: now fitted
Other:
- note added: "GNSS backup: Seiko CPH3225A 11 mF, ~10 min hot start (28 uA backup)"
- note added: "No capacitor on RESET, no load on TIMEPULSE (SAFEBOOT strap). V_BCKP fed from 3V3 via D401/R401, held up by C403."
- note removed: "GNSS backup option, DNP in v1"
- note removed: "No capacitor on RESET, no load on TIMEPULSE (SAFEBOOT strap). V_BCKP open in v1."
Changed lines of the file:
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@@
 		)
 	)
-	(text "No capacitor on RESET, no load on TIMEPULSE (SAFEBOOT strap). V_BCKP open in v1."
+	(text "No capacitor on RESET, no load on TIMEPULSE (SAFEBOOT strap). V_BCKP fed from 3V3 via D401/R401, held up by C403."
 		(exclude_from_sim no)
 		(at 25.4 41.91 0)
@@
 		)
 	)
-	(text "GNSS backup option, DNP in v1"
+	(text "GNSS backup: Seiko CPH3225A 11 mF, ~10 min hot start (28 uA backup)"
 		(exclude_from_sim no)
 		(at 96.52 48.26 0)
@@
 		(on_board yes)
 		(in_pos_files yes)
-		(dnp yes)
+		(dnp no)
 		(property "Reference" "R401"
 			(at 104.14 62.23 0)
@@
 		(on_board yes)
 		(in_pos_files yes)
-		(dnp yes)
+		(dnp no)
 		(property "Reference" "D401"
 			(at 114.3 59.69 0)
@@
 		(on_board yes)
 		(in_pos_files yes)
-		(dnp yes)
+		(dnp no)
 		(property "Reference" "C403"
 			(at 119.38 76.2 0)
@@
 			)
 		)
-		(property "Value" "0.22F 3.3V"
+		(property "Value" "11mF 3.3V"
 			(at 119.38 78.74 0)
 			(show_name no)
@@
 			)
 		)
-		(property "Footprint" ""
+		(property "Footprint" "theoros:Seiko_CPH3225A"
 			(at 116.84 77.47 0)
 			(hide yes)
@@
 			)
 		)
-		(property "Description" "Unpolarized capacitor"
+		(property "Description" "Chip EDLC for GNSS backup, polarised: pin 1 = + (V_BCKP)"
 			(at 116.84 77.47 0)
 			(hide yes)
@@
 			)
 		)
-		(property "Manufacturer" "Elna"
+		(property "Manufacturer" "Seiko Instruments"
 			(at 116.84 77.47 0)
 			(hide yes)
@@
 			)
 		)
-		(property "MPN" "DSK-3R3H224U-HL"
+		(property "MPN" "CPH3225A"
 			(at 116.84 77.47 0)
 			(hide yes)
